File: usbttl.kicad_pcb (KiCad board)
At the start: 2 copper layers, 36.8 x 38.6 mm, 23 parts, among them J1 USB_C_Receptacle, J2 Conn_01x04_Pin, J3 Conn_01x04_Pin, J4 Conn_01x04_Pin, J5 Conn_01x01_Pin, J6 Conn_01x01_Pin, J7 Conn_01x03_Pin, U1 CH340G, U2 USBLC6-2SC6, U3 AMS1117-3.3, Y1 12MHz

Commit message: Fix DRC errors
Parts:
- moved C1 1.78 mm to (113.0, 92.8)
- moved C4 1.78 mm to (113.0, 91.1)
- moved C2 1.52 mm to (110.0, 95.5)
- moved Y1 1.52 mm to (113.0, 95.5)
Routing:
- net GND: track 0.00 -> 8.98 mm, vias 0 -> 14
- net +5V: track 21.5 -> 29.8 mm
- net Net-(U1-V3): track 2.90 -> 4.73 mm
- net Net-(U1-XO): track 8.38 -> 9.44 mm
- net Net-(U1-XI): track 5.43 -> 6.27 mm
Changed lines of the file:
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@@
       (rotate (xyz 0 0 0))
-    )
-    (model "${KIPRJMOD}/step/USB_type_C_smd_12p.stp"
-      (offset (xyz 0 2.5 0))
-      (scale (xyz 1 1 1))
-      (rotate (xyz -90 0 -180))
     )
   )
@@
   )
   (footprint "Capacitor_SMD:C_0603_1608Metric" (layer "F.Cu")
-    (at 114.808 92.71 180)
+    (at 113.03 92.837 180)
     (descr "Capacitor SMD 0603 (1608 Metric), square (rectangular) end terminal, IPC_7351 nominal, (Body size source: IPC-SM-782 page 76, https://www.pcb-3d.com/wordpress/wp-content/uploads/ipc-sm-782a_amendment_1_and_2.pdf), generated with kicad-footprint-generator")
     (tags "capacitor")
@@
     (property "ki_keywords" "cap capacitor")
     (attr smd)
-    (fp_text reference "C3" (at 0 1.524) (layer "F.SilkS")
+    (fp_text reference "C3" (at 0 -1.397) (layer "F.SilkS")
         (effects (font (size 1 1) (thickness 0.15)))
     )
@@
   )
   (footprint "Capacitor_SMD:C_0603_1608Metric" (layer "F.Cu")
-    (at 114.808 90.932 180)
+    (at 113.03 91.059 180)
     (descr "Capacitor SMD 0603 (1608 Metric), square (rectangular) end terminal, IPC_7351 nominal, (Body size source: IPC-SM-782 page 76, https://www.pcb-3d.com/wordpress/wp-content/uploads/ipc-sm-782a_amendment_1_and_2.pdf), generated with kicad-footprint-generator")
     (tags "capacitor")
@@
   )
   (footprint "Crystal:Crystal_SMD_3225-4Pin_3.2x2.5mm" (layer "F.Cu")
-    (at 114.554 95.504 180)
+    (at 113.03 95.504 180)
     (descr "SMD Crystal SERIES SMD3225/4 http://www.txccrystal.com/images/pdf/7m-accuracy.pdf, 3.2x2.5mm^2 package")
     (tags "SMD SMT crystal")
@@
     (property "ki_keywords" "USB UART Serial Converter Interface")
     (attr smd)
-    (fp_text reference "U1" (at 0 6.096) (layer "F.SilkS")
+    (fp_text reference "U1" (at 0 1.27) (layer "F.SilkS")
         (effects (font (size 1 1) (thickness 0.15)))
     )
@@
     (property "ki_keywords" "diode Schottky")
     (attr smd)
-    (fp_text reference "D2" (at 0 -2 90) (layer "F.SilkS")
+    (fp_text reference "D2" (at 0 1.905 90) (layer "F.SilkS")
         (effects (font (size 1 1) (thickness 0.15)))
     )
@@
   )
   (footprint "Capacitor_SMD:C_0603_1608Metric" (layer "F.Cu")
-    (at 111.506 95.504 90)
+    (at 109.982 95.504 90)
     (descr "Capacitor SMD 0603 (1608 Metric), square (rectangular) end terminal, IPC_7351 nominal, (Body size source: IPC-SM-782 page 76, https://www.pcb-3d.com/wordpress/wp-content/uploads/ipc-sm-782a_amendment_1_and_2.pdf), generated with kicad-footprint-generator")
     (tags "capacitor")
@@
     (effects (font (size 1 1) (thickness 0.15)) (justify left bottom))
   )
+  (segment (start 113.805 94.329) (end 114.13 94.654) (width 0.25) (layer "F.Cu") (net 1))
   (segment (start 118.39 94.654) (end 118.429 94.615) (width 0.25) (layer "F.Cu") (net 1))
-  (segment (start 115.654 94.654) (end 118.39 94.654) (width 0.25) (layer "F.Cu") (net 1))
-  (segment (start 116.091 94.217) (end 115.654 94.654) (width 0.25) (layer "F.Cu") (net 1))
-  (segment (start 115.654 94.654) (end 115.654 92.893) (width 0.25) (layer "F.Cu") (net 1))
-  (segment (start 115.654 92.893) (end 115.837 92.71) (width 0.25) (layer "F.Cu") (net 1))
-  (segment (start 113.454 96.354) (end 114.89 97.79) (width 0.25) (layer "F.Cu") (net 3))
-  (segment (start 113.454 96.354) (end 111.685 96.354) (width 0.25) (layer "F.Cu") (net 3))
-  (segment (start 111.685 96.354) (end 111.506 96.533) (width 0.25) (layer "F.Cu") (net 3))
-  (segment (start 116.524 97.79) (end 118.429 95.885) (width 0.25) (layer "F.Cu") (net 3))
-  (segment (start 114.89 97.79) (end 116.524 97.79) (width 0.25) (layer "F.Cu") (net 3))
+  (segment (start 114.13 94.654) (end 118.39 94.654) (width 0.25) (layer "F.Cu") (net 1))
+  (segment (start 113.805 92.837) (end 113.805 94.329) (width 0.25) (layer "F.Cu") (net 1))
+  (segment (start 122.072 76.369) (end 122.072 76.86) (width 0.25) (layer "F.Cu") (net 2))
+  (segment (start 118.429 86.995) (end 118.034 87.39) (width 0.25) (layer "F.Cu") (net 2))
+  (segment (start 118.034 87.39) (end 115.418 87.39) (width 0.25) (layer "F.Cu") (net 2))
+  (segment (start 115.672 76.86) (end 114.554 77.978) (width 0.5) (layer "F.Cu") (net 2))
+  (segment (start 115.672 76.369) (end 115.672 76.86) (width 0.25) (layer "F.Cu") (net 2))
+  (segment (start 118.872 82.4285) (end 118.872 80.772) (width 0.5) (layer "F.Cu") (net 2))
+  (segment (start 122.072 76.86) (end 123.19 77.978) (width 0.5) (layer "F.Cu") (net 2))
+  (via (at 116.713 95.504) (size 0.8) (drill 0.4) (layers "F.Cu" "B.Cu") (free) (net 2))
+  (via (at 115.697 96.393) (size 0.8) (drill 0.4) (layers "F.Cu" "B.Cu") (free) (net 2))
+  (via (at 118.872 80.772) (size 0.8) (drill 0.4) (layers "F.Cu" "B.Cu") (free) (net 2))
+  (via (at 114.554 77.978) (size 0.8) (drill 0.4) (layers "F.Cu" "B.Cu") (free) (net 2))
+  (via (at 120.777 82.804) (size 0.8) (drill 0.4) (layers "F.Cu" "B.Cu") (free) (net 2))
+  (via (at 115.697 95.504) (size 0.8) (drill 0.4) (layers "F.Cu" "B.Cu") (free) (net 2))
+  (via (at 118.872 78.232) (size 0.8) (drill 0.4) (layers "F.Cu" "B.Cu") (free) (net 2))
+  (via (at 123.19 77.978) (size 0.8) (drill 0.4) (layers "F.Cu" "B.Cu") (free) (net 2))
+  (via (at 120.777 81.661) (size 0.8) (drill 0.4) (layers "F.Cu" "B.Cu") (free) (net 2))
+  (via (at 121.539 81.661) (size 0.8) (drill 0.4) (layers "F.Cu" "B.Cu") (free) (net 2))
+  (via (at 121.539 82.804) (size 0.8) (drill 0.4) (layers "F.Cu" "B.Cu") (free) (net 2))
+  (via (at 117.094 81.534) (size 0.8) (drill 0.4) (layers "F.Cu" "B.Cu") (free) (net 2))
+  (via (at 118.872 79.502) (size 0.8) (drill 0.4) (layers "F.Cu" "B.Cu") (free) (net 2))
+  (via (at 116.713 96.393) (size 0.8) (drill 0.4) (layers "F.Cu" "B.Cu") (free) (net 2))
+  (segment (start 118.429 95.885) (end 117.035 97.279) (width 0.25) (layer "F.Cu") (net 3))
+  (segment (start 112.855 97.279) (end 111.93 96.354) (width 0.25) (layer "F.Cu") (net 3))
+  (segment (start 117.035 97.279) (end 112.855 97.279) (width 0.25) (layer "F.Cu") (net 3))
+  (segment (start 111.93 96.354) (end 110.057 96.354) (width 0.25) (layer "F.Cu") (net 3))
+  (segment (start 110.057 96.354) (end 109.982 96.279) (width 0.25) (layer "F.Cu") (net 3))
   (segment (start 115.418 79.502) (end 115.418 82.79) (width 0.5) (layer "F.Cu") (net 4))
   (segment (start 112.268 79.502) (end 115.418 79.502) (width 0.5) (layer "F.Cu") (net 4))
   (segment (start 122.402 86.018) (end 123.379 86.995) (width 0.25) (layer "F.Cu") (net 4))
+  (segment (start 118.872 84.319249) (end 118.118751 83.566) (width 0.25) (layer "F.Cu") (net 4))
   (segment (start 121.272 76.369) (end 121.272 77.239) (width 0.5) (layer "F.Cu") (net 4))
   (segment (start 115.418 78.384) (end 115.418 79.502) (width 0.5) (layer "F.Cu") (net 4))
   (segment (start 122.402 78.369) (end 122.402 83.566) (width 0.5) (layer "F.Cu") (net 4))
+  (segment (start 118.872 84.319249) (end 119.625249 83.566) (width 0.25) (layer "F.Cu") (net 4))
   (segment (start 122.402 83.566) (end 122.402 85.344) (width 0.5) (layer "F.Cu") (net 4))
   (segment (start 116.472 76.369) (end 116.472 77.33) (width 0.5) (layer "F.Cu") (net 4))
+  (segment (start 119.625249 83.566) (end 122.402 83.566) (width 0.25) (layer "F.Cu") (net 4))
+  (segment (start 116.194 83.566) (end 115.418 82.79) (width 0.25) (layer "F.Cu") (net 4))
   (segment (start 122.402 85.344) (end 122.402 86.018) (width 0.25) (layer "F.Cu") (net 4))
+  (segment (start 118.118751 83.566) (end 116.194 83.566) (width 0.25) (layer "F.Cu") (net 4))
+  (segment (start 118.872 84.7035) (end 118.872 84.319249) (width 0.25) (layer "F.Cu") (net 4))
   (segment (start 116.472 77.33) (end 115.418 78.384) (width 0.5) (layer "F.Cu") (net 4))
   (segment (start 121.272 77.239) (end 122.402 78.369) (width 0.5) (layer "F.Cu") (net 4))
-  (segment (start 115.71 90.805) (end 115.583 90.932) (width 0.25) (layer "F.Cu") (net 5))
-  (segment (start 118.429 90.805) (end 115.71 90.805) (width 0.25) (layer "F.Cu") (net 5))
+  (segment (start 113.805 91.059) (end 118.175 91.059) (width 0.25) (layer "F.Cu") (net 5))
+  (segment (start 118.175 91.059) (end 118.429 90.805) (width 0.25) (layer "F.Cu") (net 5))
   (segment (start 121.158 95.758) (end 122.174 96.774) (width 0.25) (layer "F.Cu") (net 6))
   (segment (start 129.159 89.535) (end 131.318 87.376) (width 0.25) (layer "F.Cu") (net 6))
@@
   (via (at 117.602 97.79) (size 0.8) (drill 0.4) (layers "F.Cu" "B.Cu") (net 8))
   (via (at 106.68 88.519) (size 0.8) (drill 0.4) (layers "F.Cu" "B.Cu") (free) (net 8))
-  (segment (start 117.602 97.79) (end 117.475 97.79) (width 0.25) (layer "B.Cu") (net 8))
-  (segment (start 108.331 88.519) (end 106.68 88.519) (width 0.25) (layer "B.Cu") (net 8))
-  (segment (start 117.602 97.79) (end 108.331 88.519) (width 0.25) (layer "B.Cu") (net 8))
+  (segment (start 106.797695 88.519) (end 106.68 88.519) (width 0.25) (layer "B.Cu") (net 8))
+  (segment (start 117.602 97.79) (end 116.068695 97.79) (width 0.25) (layer "B.Cu") (net 8))
+  (segment (start 116.068695 97.79) (end 106.797695 88.519) (width 0.25) (layer "B.Cu") (net 8))
   (segment (start 100.965 95.25) (end 106.68 89.535) (width 0.25) (layer "F.Cu") (net 9))
   (segment (start 119.38 103.124) (end 120.65 104.394) (width 0.25) (layer "F.Cu") (net 9))
@@
   (segment (start 119.622 82.2285) (end 119.822 82.4285) (width 0.25) (layer "F.Cu") (net 25))
   (zone (net 2) (net_name "GND") (layer "F.Cu") (hatch edge 0.5)
-    (connect_pads (clearance 0.5))
+    (connect_pads (clearance 0.25))
     (min_thickness 0.25) (filled_areas_thickness no)
     (fill yes (thermal_gap 0.5) (thermal_bridge_width 0.5))
@@
   (zone (net 2) (net_name "GND") (layer "B.Cu") (hatch edge 0.5)
     (priority 1)
-    (connect_pads (clearance 0.5))
+    (connect_pads (clearance 0.25))
     (min_thickness 0.25) (filled_areas_thickness no)
     (fill yes (thermal_gap 0.5) (thermal_bridge_width 0.5))

Commit message: reorganize files
Parts:
- U2: footprint Package_TO_SOT_SMD:SOT-23-6 -> Package_TO_SOT_SMD:SOT-666
Routing:
- net GND: track 8.98 -> 7.32 mm
- net USB_D+: track 9.65 -> 8.95 mm
- net Net-(J1-D--PadA7): track 9.00 -> 8.38 mm
