File: usbttl.kicad_sch (KiCad schematic)
At the start: 23 parts, among them J1 USB_C_Receptacle, J2 Conn_01x04_Pin, J3 Conn_01x04_Pin, J4 Conn_01x04_Pin, J5 Conn_01x01_Pin, J6 Conn_01x01_Pin, J7 Conn_01x03_Pin, U1 CH340G, U2 USBLC6-2SC6, U3 AMS1117-3.3, Y1 12MHz

Commit message: BOM and update parts
Parts:
- U2: LCSC Part (none) -> C2827693
- U3: LCSC Part (none) -> C6186
Changed lines of the file:
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@@
+      (effects (font (size 1.27 1.27)) hide)
+    )
+    (property "LCSC Part" "C2827693" (at 133.35 83.82 90)
       (effects (font (size 1.27 1.27)) hide)
     )
@@
       (effects (font (size 1.27 1.27)) hide)
     )
+    (property "LCSC Part" "C6186" (at 115.57 102.87 0)
+      (effects (font (size 1.27 1.27)) hide)
+    )

Commit message: reorganize files
Parts:
- U2: footprint Package_TO_SOT_SMD:SOT-23-6 -> Package_TO_SOT_SMD:SOT-666
Changed lines of the file:
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@@
       (effects (font (size 1.27 1.27)))
     )
-    (property "Footprint" "Package_TO_SOT_SMD:SOT-23-6" (at 120.65 83.82 0)
+    (property "Footprint" "Package_TO_SOT_SMD:SOT-666" (at 120.65 83.82 0)
       (effects (font (size 1.27 1.27)) hide)
     )
